Commit message: Done with ros2_control

File: src/bot_description/urdf/camera.xacro (robot description, xacro)
@@ -53,3 +53,20 @@
         </sensor>
     </gazebo>
+    <joint name="imu_joint" type="fixed">
+        <origin xyz="0 0 0" rpy="0 0 0" />
+        <parent link="base_link"/>
+        <child link="imu_link" />
+    </joint>
+    <link name="imu_link">
+    </link>
+    <gazebo reference="imu_link">
+        <sensor name="imu" type="imu">
+        <always_on>1</always_on>
+        <update_rate>50</update_rate>
+        <visualize>true</visualize>
+        <topic>imu</topic>
+        <enable_metrics>true</enable_metrics>
+        <gz_frame_id>imu_link</gz_frame_id>
+        </sensor>
+    </gazebo>
 </robot>

File: src/bot_description/urdf/mobile_base.xacro (robot description, xacro)
@@ -111,14 +111,14 @@
         <origin xyz="${base_length * (3.0/8.0)} 0 -0.05" rpy="0 0 0" />
     </joint>
-    <joint name="right_wheel_base_joint" type="continuous">
+    <joint name="left_wheel_base_joint" type="continuous">
         <parent link="base_link" />
-        <child link="right_wheel_link" />
+        <child link="left_wheel_link" />
         <origin xyz="${-base_length * (3.0/8.0)} ${(base_width / 2.0) + (wheel_length / 2.0)} 0" rpy="0 0 0" />
         <axis xyz="0 1 0" />
         <limit lower="-1.57" upper="1.57" velocity="100" effort="100" />
     </joint>
-    <joint name="left_wheel_base_joint" type="continuous">
+    <joint name="right_wheel_base_joint" type="continuous">
         <parent link="base_link" />
-        <child link="left_wheel_link" />
+        <child link="right_wheel_link" />
         <origin xyz="${-base_length * (3.0/8.0)} ${(-base_width / 2.0) + (-wheel_length / 2.0)} 0" rpy="0 0 0" />
         <axis xyz="0 1 0" />

File: src/bot_description/urdf/mobile_base_gazebo.xacro (robot description, xacro)
@@ -7,5 +7,5 @@
     <gazebo>
     <plugin filename="gz_ros2_control-system" name="gz_ros2_control::GazeboSimROS2ControlPlugin">
-      <parameters>$(find-pkg-share bot_controller)/config/bot_controller.yaml</parameters>
+      <parameters>$(find bot_controller)/config/bot_controller.yaml</parameters>
     </plugin>
     <plugin filename="gz-sim-imu-system" name="gz::sim::systems::Imu">

File: src/bot_description/urdf/my_robot.urdf.xacro (robot description, xacro)
@@ -1,4 +1,4 @@
 <?xml version="1.0"?>
-<robot name="moving_bot_with_ii_dof_arm" xmlns:xacro="http://www.ros.org/wiki/xacro" >
+<robot name="bot" xmlns:xacro="http://www.ros.org/wiki/xacro" >
     <xacro:include filename="mobile_base.xacro" />
     <xacro:include filename="common_properties.xacro" />

Commit message: Computer Vision Code Published

File: src/bot_description/urdf/camera.xacro (robot description, xacro)
@@ -24,5 +24,5 @@
         <parent link="base_link"/>
         <child link="camera_link" />
-        <origin xyz="${base_length / 2.0 + box_length / 2.0} 0 ${base_height / 2.0}" rpy="0 0 0"/>
+        <origin xyz="${base_length / 2.0 + box_length / 2.0} 0 0.225" rpy="0 0 0"/>
     </joint>
     <gazebo reference="camera_link">
